Commit message: Sim collision fixed

File: Sim/guitar_model/guitar.urdf (robot description, URDF)
Before this commit: robot guitar, 8 links, 7 joints
Links:
- link string1: geometry collision cylinder length=0.656 radius=0.001; visual cylinder length=0.656 radius=0.0005
- link string2: geometry collision cylinder length=0.656 radius=0.001; visual cylinder length=0.656 radius=0.0005
- link string3: geometry collision cylinder length=0.656 radius=0.001; visual cylinder length=0.656 radius=0.0005
- link string4: geometry collision cylinder length=0.656 radius=0.001; visual cylinder length=0.656 radius=0.0005
- link string5: geometry collision cylinder length=0.656 radius=0.001; visual cylinder length=0.656 radius=0.0005
- link string6: geometry collision cylinder length=0.656 radius=0.001; visual cylinder length=0.656 radius=0.0005
